File: INA240.kicad_pcb (KiCad board)
At the start: 6 copper layers, 0 parts

Commit message: Save KiCad 10 design work
Snapshot of the schematic and PCB work done since the initial template
commit: AD7606C-18 ADC, 3x INA241A2 + PBV 1 mOhm shunts, MR60PW phase
connectors, LT8362 boost and LT3045-1 / LTC6655 analog supplies, project
libraries (lib/) and their sym/fp-lib-table.

.gitignore now excludes local history, SpinRender working files, the
stray .step export and Component Search Engine download leftovers.

Co-Authored-By: Claude Opus 5.5 <noreply@anthropic.com>
Parts:
- added C1: 0.1µF, Capacitor_SMD:C_0603_1608Metric, B.Cu at (153.2, 97.1)
- added C10: 1µF, Capacitor_SMD:C_0603_1608Metric, B.Cu at (153.1, 86.9)
- added C11: 4.7µF, Capacitor_SMD:C_0603_1608Metric, F.Cu at (140.3, 57.2)
- added C12: 10µF, Capacitor_SMD:C_0603_1608Metric, F.Cu at (149.3, 61.2)
- added C13: 10µF, Capacitor_SMD:C_0805_2012Metric, F.Cu at (148.2, 51.6)
- added C14: 10µF, Capacitor_SMD:C_0805_2012Metric, F.Cu at (148.2, 49.8)
- added C15: 10µF, Capacitor_SMD:C_0805_2012Metric, F.Cu at (148.2, 56.3)
- added C16: T491B475K016AT, T491B475K016AT:T491B, F.Cu at (-40.1, 77.8)
- added C17: 0.1µF, Capacitor_SMD:C_0603_1608Metric, B.Cu at (153.2, 80.4)
- added C18: 1µF, Capacitor_SMD:C_0603_1608Metric, B.Cu at (153.2, 78.9)
- added C19: 10µF, Capacitor_SMD:C_0805_2012Metric, F.Cu at (148.2, 58.1)
- added C2: 0.1µF, Capacitor_SMD:C_0603_1608Metric, B.Cu at (153.1, 88.4)
- added C20: 100nF, Capacitor_SMD:C_0603_1608Metric, F.Cu at (173.5, 61.0)
- added C21: 100nF, Capacitor_SMD:C_0603_1608Metric, F.Cu at (166.0, 48.2)
- added C22: 4.7µF, Capacitor_SMD:C_0603_1608Metric, F.Cu at (-76.0, 71.2)
- added C23: 100nF, Capacitor_SMD:C_0603_1608Metric, F.Cu at (-76.0, 74.5)
- added C24: 10 nF X7R 0603, Capacitor_SMD:C_0603_1608Metric, F.Cu at (-76.0, 77.9)
- added C25: 1nF C0G, Capacitor_SMD:C_0603_1608Metric, F.Cu at (170.8, 66.3)
- added C26: 1 nF X7R 0603, Capacitor_SMD:C_0603_1608Metric, F.Cu at (-76.0, 81.2)
- added C27: 1µF, Capacitor_SMD:C_0603_1608Metric, F.Cu at (-70.0, 67.8)
- added C28: 4,7 pF C0G 0603, Capacitor_SMD:C_0603_1608Metric, F.Cu at (-70.0, 71.2)
- added C29: 1nF C0G, Capacitor_SMD:C_0603_1608Metric, F.Cu at (164.8, 66.3)
- added C30: 22 µF X7R 1206, Capacitor_SMD:C_1206_3216Metric_Pad1.33x1.80mm_HandSolder, F.Cu at (-70.0, 74.5)
- added C31: 180 pF C0G/NP0, 50 V, 0603, Capacitor_SMD:C_0603_1608Metric, F.Cu at (167.8, 66.3)
- added C32: 180 pF C0G/NP0, 50 V, 0603, Capacitor_SMD:C_0603_1608Metric, F.Cu at (161.9, 66.3)
- added C33: 1nF C0G, Capacitor_SMD:C_0603_1608Metric, F.Cu at (158.9, 66.3)
- added C34: 180 pF C0G/NP0, 50 V, 0603, Capacitor_SMD:C_0603_1608Metric, F.Cu at (155.9, 66.3)
- added C35: 100nF, Capacitor_SMD:C_0603_1608Metric, F.Cu at (157.1, 61.2)
- added C36: 1uF, Capacitor_SMD:C_0603_1608Metric, F.Cu at (157.0, 56.5)
- added C37: 1uF, Capacitor_SMD:C_0603_1608Metric, F.Cu at (157.0, 53.5)
- added C38: 100nF, Capacitor_SMD:C_0603_1608Metric, F.Cu at (157.0, 55.0)
- added C39: 10µF, Capacitor_SMD:C_0805_2012Metric, F.Cu at (156.8, 59.5)
- added C41: 100nF, Capacitor_SMD:C_0603_1608Metric, F.Cu at (157.0, 57.9)
- added C5: 1µF, Capacitor_SMD:C_0603_1608Metric, B.Cu at (153.2, 95.6)
- added C8: 10µF, Capacitor_SMD:C_0603_1608Metric, F.Cu at (149.3, 54.7)
- added C9: 4.7µF, Capacitor_SMD:C_0603_1608Metric, F.Cu at (140.3, 50.8)
- added D2: PMEG2020EH, Diode_SMD:D_SOD-123F, F.Cu at (-43.6, 110.5)
- added G***: LOGO, LOGO, F.Cu at (130.6, 55.0)
- added H1: MountingHole_Pad, MountingHole:MountingHole_3.2mm_M3_Pad_Via, F.Cu at (177.5, 75.0)
- added H2: MountingHole_Pad, MountingHole:MountingHole_3.2mm_M3_Pad_Via, F.Cu at (177.5, 46.0)
- added H3: MountingHole_Pad, MountingHole:MountingHole_3.2mm_M3_Pad_Via, F.Cu at (119.4, 75.0)
- added H4: MountingHole_Pad, MountingHole:MountingHole_3.2mm_M3_Pad_Via, F.Cu at (119.4, 46.0)
- added IC1: AD7606C-18BSTZ, AD7606C-18BSTZ:QFP50P1200X1200X160-64N, F.Cu at (165.2, 56.5)
- added IC2: INA241A2IDGKR, LTC6655LNBHMS8-2.5#PBF:SOP65P490X110-8N, B.Cu at (148.5, 80.0)
- added IC3: LTC6655LNBHMS8-2.5#PBF, LTC6655LNBHMS8-2.5#PBF:SOP65P490X110-8N, F.Cu at (143.2, 60.2)
- added IC4: INA241A2IDGKR, LTC6655LNBHMS8-2.5#PBF:SOP65P490X110-8N, B.Cu at (148.5, 88.0)
- added IC5: LT8362EMSE#PBF, LT8362EMSE#PBF:LT8362EMSEPBF, F.Cu at (-49.3, 112.4)
- added IC6: INA241A2IDGKR, LTC6655LNBHMS8-2.5#PBF:SOP65P490X110-8N, B.Cu at (148.5, 96.7)
- added IC7: LTC6655BHMS8-5#PBF, LTC6655LNBHMS8-2.5#PBF:SOP65P490X110-8N, F.Cu at (143.2, 53.7)
- added IC8: LT3045EDD-1#TRPBF, LT3045EDD-1#TRPBF:SON45P300X300X80-13N-D, F.Cu at (143.2, 50.4)
- added IC9: LT3045EDD-1#TRPBF, LT3045EDD-1#TRPBF:SON45P300X300X80-13N-D, F.Cu at (143.2, 56.9)
- added J1: MR60PW, MR60PW:MR60PW, F.Cu at (132.2, 84.8)
- added J2: MR60PW, MR60PW:MR60PW, F.Cu at (164.8, 95.8)
- added L1: 744373965022, 744373965022:INDPM135125X620N, F.Cu at (-49.1, 102.7)
- added R1: PBV-R001-F1-1.0, PBV-R001-F1-1.0:PBVR001F110, F.Cu at (139.6, 82.3)
- added R11: 1kΩ, Resistor_SMD:R_0603_1608Metric, F.Cu at (147.1, 60.5)
- added R12: 49.9kΩ, Resistor_SMD:R_0603_1608Metric, F.Cu at (149.3, 59.8)
- added R13: 33Ω, Resistor_SMD:R_0603_1608Metric, F.Cu at (170.0, 68.5)
- added R14: 49.9kΩ, Resistor_SMD:R_0603_1608Metric, F.Cu at (149.3, 53.2)
- added R15: 9.1kΩ, Resistor_SMD:R_0603_1608Metric, F.Cu at (171.5, 68.5)
- added R16: 9.1kΩ, Resistor_SMD:R_0603_1608Metric, F.Cu at (165.6, 68.5)
- added R17: 33Ω, Resistor_SMD:R_0603_1608Metric, F.Cu at (164.1, 68.5)
- added R18: 9.1kΩ, Resistor_SMD:R_0603_1608Metric, F.Cu at (159.7, 68.5)
- added R19: 9.1kΩ, Resistor_SMD:R_0603_1608Metric, F.Cu at (168.6, 68.5)
- added R2: 20kΩ, Resistor_SMD:R_0603_1608Metric, F.Cu at (-53.6, 83.6)
- added R20: 9.1kΩ, Resistor_SMD:R_0603_1608Metric, F.Cu at (162.6, 68.5)
- added R21: 33Ω, Resistor_SMD:R_0603_1608Metric, F.Cu at (158.2, 68.5)
- added R22: 9.1kΩ, Resistor_SMD:R_0603_1608Metric, F.Cu at (156.7, 68.5)
- added R27: 40.2kΩ, Resistor_SMD:R_0805_2012Metric, B.Cu at (150.3, 84.2)
- added R28: 10kΩ, Resistor_SMD:R_0805_2012Metric, B.Cu at (146.9, 84.2)
- added R3: 36,5kΩ, Resistor_SMD:R_0603_1608Metric, F.Cu at (-45.8, 84.2)
- added R31: 40.2kΩ, Resistor_SMD:R_0805_2012Metric, B.Cu at (150.2, 92.2)
- added R32: 10kΩ, Resistor_SMD:R_0805_2012Metric, B.Cu at (146.8, 92.2)
- added R35: 40.2kΩ, Resistor_SMD:R_0805_2012Metric, B.Cu at (150.2, 100.8)
- added R36: 10kΩ, Resistor_SMD:R_0805_2012Metric, B.Cu at (146.8, 100.8)
- added R4: PBV-R001-F1-1.0, PBV-R001-F1-1.0:PBVR001F110, F.Cu at (139.6, 90.3)
- added R5: 1MΩ, Resistor_SMD:R_0603_1608Metric, F.Cu at (-42.1, 113.2)
- added R6: 365kΩ, Resistor_SMD:R_0603_1608Metric, F.Cu at (-45.0, 115.4)
- added R7: PBV-R001-F1-1.0, PBV-R001-F1-1.0:PBVR001F110, F.Cu at (139.6, 99.0)
- added R8: 1kΩ, Resistor_SMD:R_0603_1608Metric, F.Cu at (147.1, 54.0)
- added Re1: 1kΩ, Resistor_SMD:R_0603_1608Metric, F.Cu at (161.1, 68.5)
- added Re2: 1kΩ, Resistor_SMD:R_0603_1608Metric, F.Cu at (167.1, 68.5)
- added Re3: 1kΩ, Resistor_SMD:R_0603_1608Metric, F.Cu at (155.2, 68.5)
Routing:
- net GND: track 0.00 -> 159.1 mm, vias 0 -> 379
- net Net-(R35-Pad2): track 0.00 -> 38.7 mm, vias 0 -> 1
- net SNG-A3N: track 0.00 -> 37.7 mm, vias 0 -> 1
- net Net-(R31-Pad2): track 0.00 -> 35.0 mm, vias 0 -> 1
- net SNG-A2N: track 0.00 -> 33.1 mm, vias 0 -> 1
- net Net-(R27-Pad2): track 0.00 -> 31.5 mm, vias 0 -> 1
- net SNG-A1N: track 0.00 -> 27.8 mm, vias 0 -> 1
- net +2.5VA: track 0.00 -> 16.1 mm, vias 0 -> 19
- net SNG-V3+: track 0.00 -> 11.1 mm
- net SNG-V3-: track 0.00 -> 9.94 mm
- net SNG-1G: track 0.00 -> 8.98 mm
- net SNG-3F: track 0.00 -> 8.85 mm
- net SNG-3G: track 0.00 -> 7.68 mm
- net SNG-1F: track 0.00 -> 7.59 mm
- net SNG-V1-: track 0.00 -> 7.30 mm
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- added copper zone on F.Cu, net +2.5VA
- added copper zone on In2.Cu, net +2.5VA
- added copper zone on B.Cu, net +5VA
- added copper zone on F.Cu, net +5VA
- added copper zone on In2.Cu, net +5VA
- added copper zone on F.Cu, net +6V
- added copper zone on B.Cu, net GND
- added copper zone on F.Cu, net GND
- added copper zone on In1.Cu, net GND
- added copper zone on In2.Cu, net GND
- added copper zone on B.Cu, net IN-A
- added copper zone on F.Cu, net IN-A
- added copper zone on In1.Cu, net IN-A
- added copper zone on In2.Cu, net IN-A
- added copper zone on B.Cu, net IN-B
- added copper zone on F.Cu, net IN-B
- added copper zone on In1.Cu, net IN-B
- added copper zone on In2.Cu, net IN-B
- added copper zone on B.Cu, net IN-C
- added copper zone on F.Cu, net IN-C
- added copper zone on In1.Cu, net IN-C
- added copper zone on In2.Cu, net IN-C
- added copper zone on F.Cu, net Net-(IC1-REFCAPA)
- added copper zone on F.Cu, net Net-(IC1-REGCAP_1)
- added copper zone on F.Cu, net Net-(IC1-REGCAP_2)
- added copper zone on F.Cu, net Net-(IC3-NR)
- added copper zone on F.Cu, net Net-(IC7-VOUT_F)
- added copper zone on F.Cu, net Net-(IC8-SET)
- added copper zone on F.Cu, net Net-(IC9-SET)
- added copper zone on B.Cu, net OUT-A
- added copper zone on F.Cu, net OUT-A
- added copper zone on In1.Cu, net OUT-A
- added copper zone on In2.Cu, net OUT-A
- added copper zone on B.Cu, net OUT-B
- added copper zone on F.Cu, net OUT-B
- added copper zone on In1.Cu, net OUT-B
- added copper zone on In2.Cu, net OUT-B
- added copper zone on B.Cu, net OUT-C
- added copper zone on F.Cu, net OUT-C
- added copper zone on In1.Cu, net OUT-C
- added copper zone on In2.Cu, net OUT-C
Other:
- board outline added: 65 x 59.5 mm
- copper layers 6 -> 4
- board text added: "10kΩ"
- board text added: "2.5V"
- board text added: "40.2kΩ"
- board text added: "5V"
- board text added: "A"
- board text added: "B"
- board text added: "C"
- board text added: "FILTRE"
- board text added: "INA241A2"
- board text added: "INPUT"
- board text added: "LTC6655"
- board text added: "OUTPUT"
- board text added: "Phase A"
- board text added: "Phase B"
- board text added: "Phase C"
