File: PhaseSense-8586.kicad_pcb (KiCad board)
At the start: 4 copper layers, 65 x 59.5 mm, 83 parts, among them IC1 AD7606C-18BSTZ, IC2 INA241A2IDGKR, IC3 LTC6655LNBHMS8-2.5#PBF, IC4 INA241A2IDGKR, IC5 LT8362EMSE#PBF, IC6 INA241A2IDGKR, IC7 LTC6655BHMS8-5#PBF, IC8 LT3045EDD-1#TRPBF, IC9 LT3045EDD-1#TRPBF, J1 MR60PW, J2 MR60PW

Commit message: Fix the +2.5VA reference, add XT60PW-M connectors, predict measurement quality
- IC3: LTC6655LN-2.5 replaced by the standard LTC6655-2.5, pin 6 is now
  VOUT_S tied to VOUT_F (the LN version has NR on that pin)
- R12: 49.9k -> 24.9k on the SET pin of IC9, +2.5VA = 2.500 V instead of
  2.549 V; both points removed from the README design review
- J5, J6: two Amass XT60PW-M added on the Connectors sheet and on the PCB,
  with symbol, footprint and 3D model in lib/. Their power pins are not
  wired yet
- Simulations 07 (ESC PWM waveforms through both channels) and 08 (Monte
  Carlo on the tolerances), analysed by measurement_quality.py into
  measurement_quality.md; plot style shared in plotstyle.py
- Simulations 01, 02, 04, results.md and their figures redone for the
  corrected rail
- README, README template and CHANGELOG updated; all sheets re-saved from
  KiCad

Co-Authored-By: Claude Opus 5.5 <noreply@anthropic.com>
Parts:
- added J5: XT60PW-M, PhaseSense-8586:XT60PWM, F.Cu at (132.2, 35.2)
- added J6: XT60PW-M, PhaseSense-8586:XT60PWM, F.Cu at (164.6, 27.2)
- IC3: value LTC6655LNBHMS8-2.5#PBF -> LTC6655BHMS8-2.5#PBF
- R12: value 49.9kΩ -> 24.9kΩ
