File: PhaseSense-8586.kicad_sch (KiCad schematic)
At the start: 0 parts

Commit message: Fill template pages: block diagram, power sequencing, cover notes, architecture
- Block Diagram redrawn from the real design: phase path (MR60PW, shunts),
  current and voltage channels with their gains and bandwidths, AD7606C-18,
  power chain, target specifications
- Power - Sequencing: start-up curves taken from the LTspice simulations
  (boost soft-start, analog rails) and rail table with sources, levels
  and timings
- Cover page: real design notes instead of the template examples
- Project Architecture: power-supply block documented, contiguous page
  numbers (Power Supply is page 6)
- Revision History: one column fed by the [Unreleased] changelog section
- sheet titles shortened so they fit the cover-page index: INA241 - Phase
  Sensing, Power Supply - Analog Rails

Sheet-level polylines carry no fill attribute (KiBot schematic reader).

Co-Authored-By: Claude Opus 5.5 <noreply@anthropic.com>
Other:
- note added: "3-phase current and voltage sensing: INA241A2 + AD7606C-18"
- note removed: "Comment"
Changed lines of the file:
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@@
 		)
 	)
-	(text "Comment"
+	(text "3-phase current and voltage sensing: INA241A2 + AD7606C-18"
 		(exclude_from_sim no)
 		(at 222.25 177.8 0)
@@
 		)
 	)
-	(text_box "DESIGN NOTE:\nExample text for cautionary design notes."
+	(text_box "DESIGN NOTE:\nAD7606C digital pins and +3.3V input not wired yet."
 		(exclude_from_sim no)
 		(at 96.52 258.445 0)
@@
 		)
 	)
-	(text_box "DESIGN NOTE:\nExample text for debug notes."
+	(text_box "DESIGN NOTE:\nNo Power-Good: rails within 0.1 % after 71 ms."
 		(exclude_from_sim no)
 		(at 61.595 258.445 0)
@@
 		)
 	)
-	(text_box "DESIGN NOTE:\nExample text for critical design notes."
+	(text_box "DESIGN NOTE:\n+2.5VA: IC3 pin 6 (NR) tied to VOUT, R12 = 49.9k. See README."
 		(exclude_from_sim no)
 		(at 131.445 258.445 0)
@@
 		)
 	)
-	(text_box "LAYOUT NOTE:\nExample text for critical layout guidelines."
+	(text_box "LAYOUT NOTE:\nKelvin-route the shunt sense pads to each INA241."
 		(exclude_from_sim no)
 		(at 166.37 258.445 0)
@@
 		)
 	)
-	(text_box "DESIGN NOTE:\nExample text for informational design notes."
+	(text_box "DESIGN NOTE:\nCurrent: 2.5 V - 20 mV/A x I(J1->J2). Voltage: 0.198 V/V."
 		(exclude_from_sim no)
 		(at 26.67 258.445 0)

Commit message: Fix the +2.5VA reference, add XT60PW-M connectors, predict measurement quality
- IC3: LTC6655LN-2.5 replaced by the standard LTC6655-2.5, pin 6 is now
  VOUT_S tied to VOUT_F (the LN version has NR on that pin)
- R12: 49.9k -> 24.9k on the SET pin of IC9, +2.5VA = 2.500 V instead of
  2.549 V; both points removed from the README design review
- J5, J6: two Amass XT60PW-M added on the Connectors sheet and on the PCB,
  with symbol, footprint and 3D model in lib/. Their power pins are not
  wired yet
- Simulations 07 (ESC PWM waveforms through both channels) and 08 (Monte
  Carlo on the tolerances), analysed by measurement_quality.py into
  measurement_quality.md; plot style shared in plotstyle.py
- Simulations 01, 02, 04, results.md and their figures redone for the
  corrected rail
- README, README template and CHANGELOG updated; all sheets re-saved from
  KiCad

Co-Authored-By: Claude Opus 5.5 <noreply@anthropic.com>
Changed lines of the file:
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@@
 	(title_block
 		(title "PhaseSense-8586 - PHASETRACKER")
-		(date "2026-10-05")
+		(date "2026-10-06")
 		(rev "${REVISION}")
 		(company "${COMPANY}")
@@
 		)
 	)
-	(text_box "DESIGN NOTE:\n+2.5VA: IC3 pin 6 (NR) tied to VOUT, R12 = 49.9k. See README."
+	(text_box "DESIGN NOTE:\n+2.5VA: R12 = 49.9k gives 2.55 V, 24.9k gives 2.50 V. See README."
 		(exclude_from_sim no)
 		(at 131.445 258.445 0)
