File: OPEN_PHASE.kicad_pcb (KiCad board)
At the start: 4 copper layers, 65 x 59.5 mm, 85 parts, among them IC1 AD7606C-18BSTZ, IC2 INA241A2IDGKR, IC3 LTC6655BHMS8-2.5#PBF, IC4 INA241A2IDGKR, IC5 LT8362EMSE#PBF, IC6 INA241A2IDGKR, IC7 LTC6655BHMS8-5#PBF, IC8 LT3045EDD-1#TRPBF, IC9 LT3045EDD-1#TRPBF, J1 MR60PW, J2 MR60PW, J5 XT60PW-M, J6 XT60PW-M

Commit message: Rename the project to OPEN_PHASE
PhaseSense-8586 was named after the first parts of the design (INA240 +
ADS8586S), which are no longer on the board. OPEN_PHASE follows
OPEN_WEIGHT, the other OPEN THRUST LAB board.

- project files: OPEN_PHASE.kicad_pro / _sch / _pcb / _prl / _dru
- libraries: lib/lib_sym/OPEN_PHASE.kicad_sym and
  lib/lib_fp/OPEN_PHASE.pretty, nickname OPEN_PHASE in both tables, in
  every lib_id and in every footprint of the PCB
- project name of every symbol and sheet instance, so the reference
  designators are kept
- PROJECT_NAME and GIT_URL in the project and in kibot_main.yaml, README
  and its template, CHANGELOG, LTspice headers and their generator
- the README note now says the project was first published as
  PhaseSense-8586

The GitHub repository is now foukouda/OPEN_PHASE. The board name
PHASETRACKER is unchanged. The netlist, ERC and DRC reports are the same
before and after the rename.

Co-Authored-By: Claude Opus 5.5 <noreply@anthropic.com>
Parts:
- C1, C10, C11, C12, C17, C18, C2, C20, C21, C22, C23, C24, C25, C26, C27, C28, C29, C31, C32, C33, C34, C35, C36, C37, C38, C41, C5, C8, C9: footprint PhaseSense-8586:C_0603_1608Metric -> OPEN_PHASE:C_0603_1608Metric
- C13, C14, C15, C19, C39: footprint PhaseSense-8586:C_0805_2012Metric -> OPEN_PHASE:C_0805_2012Metric
- C16: footprint PhaseSense-8586:T491B -> OPEN_PHASE:T491B
- C30: footprint PhaseSense-8586:C_1206_3216Metric_Pad1.33x1.80mm_HandSolder -> OPEN_PHASE:C_1206_3216Metric_Pad1.33x1.80mm_HandSolder
- D2: footprint PhaseSense-8586:D_SOD-123F -> OPEN_PHASE:D_SOD-123F
- H1, H2, H3, H4: footprint PhaseSense-8586:MountingHole_3.2mm_M3_Pad_Via -> OPEN_PHASE:MountingHole_3.2mm_M3_Pad_Via
- IC1: footprint PhaseSense-8586:QFP50P1200X1200X160-64N -> OPEN_PHASE:QFP50P1200X1200X160-64N
- IC2, IC3, IC4, IC6, IC7: footprint PhaseSense-8586:SOP65P490X110-8N -> OPEN_PHASE:SOP65P490X110-8N
- IC5: footprint PhaseSense-8586:LT8362EMSEPBF -> OPEN_PHASE:LT8362EMSEPBF
- IC8, IC9: footprint PhaseSense-8586:SON45P300X300X80-13N-D -> OPEN_PHASE:SON45P300X300X80-13N-D
- J1, J2: footprint PhaseSense-8586:MR60PW -> OPEN_PHASE:MR60PW
- J5, J6: footprint PhaseSense-8586:XT60PWM -> OPEN_PHASE:XT60PWM
- L1: footprint PhaseSense-8586:INDPM135125X620N -> OPEN_PHASE:INDPM135125X620N
- R1, R4, R7: footprint PhaseSense-8586:PBVR001F110 -> OPEN_PHASE:PBVR001F110
- R11, R12, R13, R14, R15, R16, R17, R18, R19, R2, R20, R21, R22, R3, R5, R6, R8, Re1, Re2, Re3: footprint PhaseSense-8586:R_0603_1608Metric -> OPEN_PHASE:R_0603_1608Metric
- R27, R28, R31, R32, R35, R36: footprint PhaseSense-8586:R_0805_2012Metric -> OPEN_PHASE:R_0805_2012Metric

Commit message: Smaller boost inductor, white board, openEMS and thermal simulations
- L1: Wurth 744373965022 (13.5 x 12.5 mm) -> WE-MAPI 4030 74438357022
  (2.2 uH, 4.1 x 4.1 x 3.1 mm, Isat 4.6 A at -10 %, above the 3.1 A LT8362
  switch limit). Footprint and STEP from the KiCad library, copied to lib/.
- Board: solder mask white (custom opaque #F4F4F0F5, the KiCad "White"
  preset renders pink over copper), silkscreen black. kibot_globals.yaml
  names the colours so the fabrication notes print WHITE / BLACK.
- Simulation/openEMS: inductance of the PBV shunts seen by the INA241
  inputs on the routed copper (results.md, figures in Images/Simulation).
- Simulation/Thermal: current density and temperature of the power paths.
- LTspice simulations, figures and README updated; sim07 DC bus figure.
- 3D animation (Images/OPEN_PHASE.mp4, OPEN_PHASE-spin.gif) on the white board.
- XT60PW-F footprint and model, bottom silkscreen cartouches.

Co-Authored-By: Claude Opus 5.5 <noreply@anthropic.com>
Parts:
- removed J6: XT60PW-M, OPEN_PHASE:XT60PWM
- added C3: 0.1µF, OPEN_PHASE:C_0603_1608Metric, B.Cu at (153.2, 35.8)
- added C40: 180 pF C0G/NP0, 50 V, 0603, OPEN_PHASE:C_0603_1608Metric, F.Cu at (157.2, 50.3)
- added C42: 1nF C0G, OPEN_PHASE:C_0603_1608Metric, F.Cu at (157.2, 53.3)
- added IC10: INA241A2IDGKR, OPEN_PHASE:SOP65P490X110-8N, B.Cu at (148.5, 35.4)
- added J3: XT60PW-F, OPEN_PHASE:AMASS_XT60PW-F_1x02_P7.20mm_Horizontal, F.Cu at (130.7, 30.6)
- added NT1: NetTie_2, NetTie:NetTie-2_SMD_Pad0.5mm, B.Cu at (144.2, 33.1)
- added R30: 33Ω, OPEN_PHASE:R_0603_1608Metric, F.Cu at (154.9, 52.5)
- added R31: 9.1kΩ, OPEN_PHASE:R_0603_1608Metric, F.Cu at (154.9, 54.0)
- added R32: 40.2kΩ, OPEN_PHASE:R_0805_2012Metric, B.Cu at (150.2, 40.1)
- added R33: 10kΩ, OPEN_PHASE:R_0805_2012Metric, B.Cu at (146.8, 40.1)
- added R34: 9.1kΩ, OPEN_PHASE:R_0603_1608Metric, F.Cu at (154.9, 51.0)
- added R9: PBV-R001-F1-1.0, OPEN_PHASE:PBVR001F110, F.Cu at (139.6, 37.8)
- added Re4: 1kΩ, OPEN_PHASE:R_0603_1608Metric, F.Cu at (154.9, 49.5)
- C16: value T491B475K016AT -> 1µF; footprint OPEN_PHASE:T491B -> OPEN_PHASE:C_0603_1608Metric; moved to B.Cu
- G***: moved to B.Cu
- L1: value 744373965022 -> 74438357022; footprint OPEN_PHASE:INDPM135125X620N -> OPEN_PHASE:L_Wuerth_MAPI-4030
- moved C23 211.2 mm to (133.5, 48.0), turned to 90 degrees
- moved C22 209.3 mm to (132.0, 48.0), turned to 90 degrees
- moved C24 208.0 mm to (130.9, 56.7), turned to -90 degrees
- moved C30 207.1 mm to (136.4, 57.1), turned to 90 degrees
- moved C26 206.3 mm to (127.6, 48.0), turned to 90 degrees
- moved C27 201.5 mm to (130.5, 48.0), turned to 90 degrees
- moved C16 198.1 mm to (153.2, 34.3), turned to 0 degrees
- moved C28 197.8 mm to (127.2, 56.0)
- moved L1 191.4 mm to (135.5, 52.5), turned to -90 degrees
- moved IC5 189.9 mm to (130.9, 52.4), turned to 180 degrees
- moved D2 185.5 mm to (134.0, 56.8), turned to 90 degrees
- moved R2 185.0 mm to (129.4, 56.7), turned to -90 degrees
- moved R6 183.1 mm to (127.2, 53.1), turned to 180 degrees
- moved R5 179.2 mm to (127.2, 54.5), turned to 0 degrees
- moved R3 178.6 mm to (129.1, 48.0), turned to 90 degrees
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- renumbered R13 to R15, R15 to R16, R27 to R17, R28 to R18, R17 to R20, R16 to R21, R31 to R22, R32 to R23, R20 to R24, R21 to R25, R18 to R26, R35 to R27, R36 to R28, R22 to R29, Re2 to Re1, Re1 to Re2
Connections:
- net IN-A renamed IN-U
- net IN-B renamed IN-V
- net IN-C renamed IN-W
- net OUT-A renamed OUT-U
- net OUT-C renamed OUT-W
- C16 pad 1: unconnected-(C16-+-Pad1) -> +5VA
- C16 pad 2: unconnected-(C16---Pad2) -> GND
- IC1 pad 49: SNG-V3+ -> SNG-V4+
- IC1 pad 50: SNG-V3- -> SNG-V4-
- IC1 pad 51: SNG-3F -> SNG-4F
- IC1 pad 52: SNG-3G -> SNG-4G
- IC1 pad 53: SNG-V2+ -> SNG-V3+
- IC1 pad 54: SNG-V2- -> SNG-V3-
- IC1 pad 55: SNG-2F -> SNG-3F
- IC1 pad 56: SNG-2G -> SNG-3G
- IC1 pad 57: SNG-V1+ -> SNG-V2+
- IC1 pad 58: SNG-V1- -> SNG-V2-
- IC1 pad 59: SNG-1F -> SNG-2F
- IC1 pad 60: SNG-1G -> SNG-2G
- IC1 pad 61: unconnected-(IC1-V7+-Pad61) -> SNG-V1+
- IC1 pad 62: unconnected-(IC1-V7--Pad62) -> SNG-V1-
- IC1 pad 63: unconnected-(IC1-V8+-Pad63) -> SNG-1F
- IC1 pad 64: unconnected-(IC1-V8--Pad64) -> SNG-1G
- J2 pad 2: OUT-B -> OUT-V
- J5 pad 1: unconnected-(J5-Pad1) -> GND1
- J5 pad 2: unconnected-(J5-Pad2) -> OUT-B
- R22 pad 1: OUT-B -> OUT-V
- R4 pad 4: OUT-B -> OUT-V
Routing:
- net GND: track 159.1 -> 104.3 mm, vias 379 -> 356
- net +2.5VA: track 16.1 -> 41.4 mm, vias 19 -> 22
- net SNG-A4N: track 0.00 -> 25.0 mm, vias 0 -> 1
- net Net-(R32-Pad2): track 0.00 -> 18.5 mm, vias 0 -> 1
- net Net-(R27-Pad2): track 38.7 -> 54.0 mm
- net SNG-V4+: track 0.00 -> 12.6 mm
- net SNG-V4-: track 0.00 -> 12.1 mm
- net SNG-A3N: track 37.7 -> 49.8 mm
- net SNG-4F: track 0.00 -> 11.2 mm
- net +6V: track 0.00 -> 11.2 mm, vias 8 -> 5
- net SNG-4G: track 0.00 -> 10.5 mm
- net SNG-A1N: track 27.8 -> 17.8 mm
- net Net-(R17-Pad2): track 31.5 -> 24.4 mm
- net SNG-1F: track 7.59 -> 11.6 mm
- net SNG-V1+: track 6.27 -> 9.93 mm
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- added copper zone on F.Cu, net +3.3V
- added copper zone on F.Cu, net /Project Architecture/Power_Supply/FBX
- added copper zone on B.Cu, net GND1
- added copper zone on F.Cu, net GND1
- added copper zone on In1.Cu, net GND1
- added copper zone on In2.Cu, net GND1
- added copper zone on B.Cu, net IN-B
- added copper zone on F.Cu, net IN-B
- added copper zone on In1.Cu, net IN-B
- added copper zone on In2.Cu, net IN-B
- added copper zone on F.Cu, net Net-(D2-A)
- added copper zone on B.Cu, net OUT-V
- added copper zone on F.Cu, net OUT-V
- added copper zone on In1.Cu, net OUT-V
- added copper zone on In2.Cu, net OUT-V
Other:
- board size 65 x 59.5 mm -> 65 x 77.5 mm
- board text added: "BATTERIE"
- board text added: "BATTERIE IN"
- board text added: "BATTERIE OUT"
- board text added: "MOTOR IN"
- board text added: "MOTOR OUT"
- board text added: "Phase U"
- board text added: "Phase V"
- board text added: "Phase W"
- board text added: "U"
- board text added: "V"
- board text added: "W"
- board text removed: "A"
- board text removed: "B"
- board text removed: "C"
- board text removed: "INPUT"
- board text removed: "OUTPUT"
- board text removed: "Phase A"
- board text removed: "Phase B"
- board text removed: "Phase C"

Commit message: Wire the AD7606C-18 digital side to host header J4, add test points
- AD7606C-18: software mode (OS0-2 high), serial (PAR/SER SEL high),
  REF SELECT low; CONVST, BUSY, RESET, CS, SCLK, SDI, FRSTDATA and
  DOUTA-D to J4 (2x8 pin header 2.54 mm, horizontal), +3.3V on J4 pin 1
- AD7606C-18 AGND pin 26 and REFGND pin 46 on GND
- Test points TP1-TP16: rails, INA241 outputs, CONVST, BUSY
- Nets renamed SHUNT_*, INA_*, ADC_*; net colours in the project
- LT3045-1 footprint: thermal vias numbered as exposed pad 13
- PCB updated from the schematic; ADC_* digital nets not routed yet
- README template / CHANGELOG: status, J4 pinout, design review 1 and 2
  fixed, new finding 9 (VDRIVE above AVCC + 0.3 V at power-up),
  4 channels / 8 ADC inputs

Co-Authored-By: Claude Opus 5.5 <noreply@anthropic.com>
Parts:
- added J4: PinHeader_2x08, OPEN_PHASE:PinHeader_2x08_P2.54mm_Horizontal, F.Cu at (122.7, 69.5)
- added TP1: TestPoint, OPEN_PHASE:TestPoint_Pad_D1.5mm, B.Cu at (84.8, 66.9)
- added TP10: TestPoint, OPEN_PHASE:TestPoint_Pad_D1.5mm, B.Cu at (90.3, 61.4)
- added TP11: TestPoint, OPEN_PHASE:TestPoint_Pad_D1.5mm, B.Cu at (90.3, 64.9)
- added TP12: TestPoint, OPEN_PHASE:TestPoint_Pad_D1.5mm, B.Cu at (90.3, 68.5)
- added TP13: TestPoint, OPEN_PHASE:TestPoint_Pad_D1.5mm, B.Cu at (90.3, 72.0)
- added TP14: TestPoint, OPEN_PHASE:TestPoint_Pad_D1.5mm, B.Cu at (79.2, 66.9)
- added TP15: TestPoint, OPEN_PHASE:TestPoint_Pad_D1.5mm, B.Cu at (71.6, 60.2)
- added TP16: TestPoint, OPEN_PHASE:TestPoint_Pad_D1.5mm, B.Cu at (71.6, 63.8)
- added TP2: TestPoint, OPEN_PHASE:TestPoint_Pad_D1.5mm, B.Cu at (84.8, 70.5)
- added TP3: TestPoint, OPEN_PHASE:TestPoint_Pad_D1.5mm, B.Cu at (84.8, 57.8)
- added TP4: TestPoint, OPEN_PHASE:TestPoint_Pad_D1.5mm, B.Cu at (84.8, 61.4)
- added TP5: TestPoint, OPEN_PHASE:TestPoint_Pad_D1.5mm, B.Cu at (81.2, 57.8)
- added TP6: TestPoint, OPEN_PHASE:TestPoint_Pad_D1.5mm, B.Cu at (81.2, 61.4)
- added TP7: TestPoint, OPEN_PHASE:TestPoint_Pad_D1.5mm, B.Cu at (77.7, 57.8)
- added TP8: TestPoint, OPEN_PHASE:TestPoint_Pad_D1.5mm, B.Cu at (77.7, 61.4)
- added TP9: TestPoint, OPEN_PHASE:TestPoint_Pad_D1.5mm, B.Cu at (90.3, 57.8)
- moved G*** 42.6 mm to (169.6, 54.0)
- moved IC3 6.20 mm to (126.3, 67.1)
- moved C12 6.20 mm to (125.2, 73.3)
- moved C8 6.20 mm to (131.8, 73.3)
- moved IC7 6.20 mm to (132.8, 67.1)
- moved R11 6.20 mm to (126.0, 71.1)
- moved R12 6.20 mm to (126.8, 73.3)
- moved R14 6.20 mm to (133.3, 73.3)
- moved R8 6.20 mm to (132.5, 71.0)
- moved C11 6.20 mm to (129.2, 64.3)
- moved C13 6.20 mm to (134.9, 72.2)
- moved C14 6.20 mm to (136.7, 72.2)
- moved C15 6.20 mm to (130.2, 72.2)
- moved C19 6.20 mm to (128.4, 72.2)
- moved C9 6.20 mm to (135.8, 64.3)
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Connections:
- net IN-1 renamed SHUNT_U-
- net IN-2 renamed SHUNT_V-
- net IN-3 renamed SHUNT_W-
- net IN-4 renamed SHUNT_BAT-
- net OUT-1 renamed SHUNT_U+
- net OUT-2 renamed SHUNT_V+
- net OUT-3 renamed SHUNT_W+
- net OUT-4 renamed SHUNT_BAT+
- net SNG-1F renamed ADC_U_I+
- net SNG-1G renamed ADC_U_I-
- net SNG-2F renamed ADC_V_I+
- net SNG-2G renamed ADC_V_I-
- net SNG-3F renamed ADC_W_I+
- net SNG-3G renamed ADC_W_I-
- net SNG-4F renamed ADC_BAT_I+
- net SNG-4G renamed ADC_BAT_I-
- net SNG-A1N renamed INA_U
- net SNG-A2N renamed INA_V
- net SNG-A3N renamed INA_W
- net SNG-A4N renamed INA_BAT
- net SNG-V1+ renamed ADC_U_V+
- net SNG-V1- renamed ADC_U_V-
- net SNG-V2+ renamed ADC_V_V+
- net SNG-V2- renamed ADC_V_V-
- net SNG-V3+ renamed ADC_W_V+
- net SNG-V3- renamed ADC_W_V-
- net SNG-V4+ renamed ADC_BAT_V+
- net SNG-V4- renamed ADC_BAT_V-
- IC1 pad 10: unconnected-(IC1-~{WR}-Pad10) -> +3.3V
- IC1 pad 11: unconnected-(IC1-RESET-Pad11) -> ADC_RESET
- IC1 pad 12: unconnected-(IC1-~{RD}/SCLK-Pad12) -> ADC_SCLK
- IC1 pad 13: unconnected-(IC1-~{CS}-Pad13) -> ADC_~{CS}
- IC1 pad 14: unconnected-(IC1-BUSY-Pad14) -> ADC_BUSY
- IC1 pad 15: unconnected-(IC1-FRSTDATA-Pad15) -> ADC_FRSTDATA
- IC1 pad 16: unconnected-(IC1-DB2-Pad16) -> GND
- IC1 pad 17: unconnected-(IC1-DB3-Pad17) -> GND
- IC1 pad 18: unconnected-(IC1-DB4-Pad18) -> GND
- IC1 pad 24: unconnected-(IC1-DB9/DOUTA-Pad24) -> ADC_DOUTA
- IC1 pad 25: unconnected-(IC1-DB10/DOUTB-Pad25) -> ADC_DOUTB
- IC1 pad 26: unconnected-(IC1-AGND_2-Pad26) -> GND
- IC1 pad 27: unconnected-(IC1-DB11/DOUTC-Pad27) -> ADC_DOUTC
- IC1 pad 28: unconnected-(IC1-DB12/DOUTD-Pad28) -> ADC_DOUTD
- IC1 pad 29: unconnected-(IC1-DB13/SDI-Pad29) -> ADC_SDI
- IC1 pad 3: unconnected-(IC1-OS_0-Pad3) -> +3.3V
- IC1 pad 30: unconnected-(IC1-DB14-Pad30) -> GND
- IC1 pad 31: unconnected-(IC1-DB15-Pad31) -> GND
- IC1 pad 32: unconnected-(IC1-DB16/DB0-Pad32) -> GND
- IC1 pad 33: unconnected-(IC1-DB17/DB1-Pad33) -> GND
- IC1 pad 34: unconnected-(IC1-REF_SELECT-Pad34) -> GND
- IC1 pad 4: unconnected-(IC1-OS_1-Pad4) -> +3.3V
- IC1 pad 46: unconnected-(IC1-REFGND_2-Pad46) -> GND
- IC1 pad 5: unconnected-(IC1-OS_2-Pad5) -> +3.3V
- IC1 pad 6: unconnected-(IC1-~{PAR}/SER_SEL-Pad6) -> +3.3V
- IC1 pad 7: unconnected-(IC1-~{STBY}-Pad7) -> +3.3V
- IC1 pad 8: unconnected-(IC1-RANGE-Pad8) -> +3.3V
- IC1 pad 9: unconnected-(IC1-CONVST-Pad9) -> ADC_CONVST
Routing:
- net +2.5VA: track 41.4 -> 20.8 mm
- net GND: track 104.3 -> 104.4 mm, vias 356 -> 355
Other:
- board text added: "+3.3V"
- board text added: "BUSY"
- board text added: "CONVST"
- board text added: "CS"
- board text added: "DOUTA"
- board text added: "DOUTB"
- board text added: "DOUTC"
- board text added: "DOUTD"
- board text added: "FRSTDATA"
- board text added: "GND"
- board text added: "RESET"
- board text added: "SCLK"
- board text added: "SDI"

Commit message: Add rail indicator LEDs, test point tags and OSHW logo
- Schematic: D1, D3-D5 rail indicator LEDs on +2.5VA, +5VA, +3.3V and
  +6V. Series resistors R35 750 R, R37 1.5k, R36 3.3k, R38 4.3k: about
  1 mA each with a Wurth 150060RS75000 (red, 1.78 V at 1 mA).
- PCB F.SilkS: rail name beside each LED (Airborne 0.8 mm knockout).
- PCB B.SilkS: J4-style tags on the 10 placed test points (pill that
  wraps the pad, net name in Arial Black knockout), OSHW logo LOGO2
  (board only) next to the bottom logo.
- lib: OSHW-Logo_7.5x8mm_SilkScreen added to the project footprints.
- Images: 3D spin animation in the blue / white colours.

DRC and schematic parity counts are unchanged by the silkscreen work.

Co-Authored-By: Claude Opus 5.5 <noreply@anthropic.com>
Parts:
- removed TP1, TP13, TP14, TP2, TP7, TP8: TestPoint, OPEN_PHASE:TestPoint_Pad_D1.5mm
- added D1: LED, LED_SMD:LED_0603_1608Metric, F.Cu at (142.6, 61.6)
- added D3: LED, LED_SMD:LED_0603_1608Metric, F.Cu at (142.6, 60.2)
- added D4: LED, LED_SMD:LED_0603_1608Metric, F.Cu at (142.6, 57.4)
- added D5: LED, LED_SMD:LED_0603_1608Metric, F.Cu at (142.6, 58.8)
- added LOGO2: OSHW-Logo_7.5x8mm_SilkScreen, OPEN_PHASE:OSHW-Logo_7.5x8mm_SilkScreen, B.Cu at (158.6, 54.0)
- added R35: 33Ω, OPEN_PHASE:R_0603_1608Metric, F.Cu at (140.0, 61.6)
- added R36: 33Ω, OPEN_PHASE:R_0603_1608Metric, F.Cu at (140.0, 60.2)
- added R37: 33Ω, OPEN_PHASE:R_0603_1608Metric, F.Cu at (140.0, 57.4)
- added R38: 33Ω, OPEN_PHASE:R_0603_1608Metric, F.Cu at (140.0, 58.8)
- moved TP16 101.1 mm to (172.6, 69.2)
- moved TP15 95.9 mm to (167.0, 70.0)
- moved TP6 71.9 mm to (152.5, 52.0)
- moved TP5 71.3 mm to (152.5, 58.0)
- moved TP3 68.8 mm to (152.5, 70.0)
- moved TP4 67.8 mm to (152.5, 64.0)
- moved TP11 52.4 mm to (142.7, 65.5)
- moved TP12 50.6 mm to (140.8, 72.5)
- moved TP10 46.2 mm to (136.6, 61.1)
- moved TP9 44.9 mm to (134.4, 48.9)
Routing:
- net ADC_SCLK: track 0.00 -> 64.5 mm, vias 0 -> 1
- net ADC_SDI: track 0.00 -> 64.4 mm, vias 0 -> 1
- net ADC_DOUTD: track 0.00 -> 63.0 mm, vias 0 -> 1
- net ADC_DOUTB: track 0.00 -> 62.4 mm, vias 0 -> 1
- net ADC_DOUTC: track 0.00 -> 60.1 mm, vias 0 -> 1
- net ADC_FRSTDATA: track 0.00 -> 58.6 mm, vias 0 -> 1
- net ADC_RESET: track 0.00 -> 57.3 mm, vias 0 -> 1
- net ADC_BUSY: track 0.00 -> 56.7 mm, vias 0 -> 1
- net ADC_~{CS}: track 0.00 -> 55.2 mm, vias 0 -> 1
- net ADC_DOUTA: track 0.00 -> 53.8 mm, vias 0 -> 1
- net ADC_CONVST: track 0.00 -> 51.3 mm, vias 0 -> 1
- net +2.5VA: track 20.8 -> 29.1 mm, vias 22 -> 24
- net +3.3V: track 0.00 -> 7.64 mm, vias 1 -> 9
- net +6V: track 11.2 -> 15.1 mm, vias 5 -> 6
- net +5VA: track 0.00 -> 0.55 mm, vias 25 -> 27
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- added copper zone on In2.Cu, net +3.3V
Other:
- board text added: "+2.5VA"
- board text added: "+5VA"
- board text added: "+6V"
- board text added: "B"
- board text added: "INA BAT"
- board text added: "INA U"
- board text added: "INA V"
- board text added: "INA W"
