File: AD7606C-18 - ADC.kicad_sch (KiCad schematic)
At the start: 9 parts, among them IC1 AD7606C-18BSTZ

Commit message: Wire the AD7606C-18 digital side to host header J4, add test points
- AD7606C-18: software mode (OS0-2 high), serial (PAR/SER SEL high),
  REF SELECT low; CONVST, BUSY, RESET, CS, SCLK, SDI, FRSTDATA and
  DOUTA-D to J4 (2x8 pin header 2.54 mm, horizontal), +3.3V on J4 pin 1
- AD7606C-18 AGND pin 26 and REFGND pin 46 on GND
- Test points TP1-TP16: rails, INA241 outputs, CONVST, BUSY
- Nets renamed SHUNT_*, INA_*, ADC_*; net colours in the project
- LT3045-1 footprint: thermal vias numbered as exposed pad 13
- PCB updated from the schematic; ADC_* digital nets not routed yet
- README template / CHANGELOG: status, J4 pinout, design review 1 and 2
  fixed, new finding 9 (VDRIVE above AVCC + 0.3 V at power-up),
  4 channels / 8 ADC inputs

Co-Authored-By: Claude Opus 5.5 <noreply@anthropic.com>
Parts:
- added TP1, TP15, TP16, TP2: TestPoint, OPEN_PHASE:TestPoint_Pad_D1.5mm, symbol OPEN_PHASE:TestPoint
Connections:
- net +2.5VA: now also TP1.1
- net +3.3V: now also IC1.10 (~{WR}), IC1.3 (OS_0), IC1.4 (OS_1), IC1.5 (OS_2), IC1.6 (~{PAR}/SER_SEL), IC1.7 (~{STBY}), IC1.8 (RANGE)
- net GND: now also IC1.16 (DB2), IC1.17 (DB3), IC1.18 (DB4), IC1.26 (AGND_2), IC1.30 (DB14), IC1.31 (DB15), IC1.32 (DB16/DB0), IC1.33 (DB17/DB1), IC1.34 (REF_SELECT), IC1.46 (REFGND_2), TP2.1
- net ADC_RESET: now reaches IC1.11 (RESET)
- net ADC_SCLK: now reaches IC1.12 (~{RD}/SCLK)
- net ADC_~{CS}: now reaches IC1.13 (~{CS})
- net ADC_BUSY: now reaches IC1.14 (BUSY)
- net ADC_BUSY: now also TP16.1
- net ADC_FRSTDATA: now reaches IC1.15 (FRSTDATA)
- net ADC_DOUTA: now reaches IC1.24 (DB9/DOUTA)
- net ADC_DOUTB: now reaches IC1.25 (DB10/DOUTB)
- net ADC_DOUTC: now reaches IC1.27 (DB11/DOUTC)
- net ADC_DOUTD: now reaches IC1.28 (DB12/DOUTD)
- net ADC_SDI: now reaches IC1.29 (DB13/SDI)
- net ADC_CONVST: now reaches IC1.9 (CONVST)
- net ADC_CONVST: now also TP15.1
- net SNG-1F renamed ADC_U_I+
- net SNG-1G renamed ADC_U_I-
- net SNG-2F renamed ADC_V_I+
- net SNG-2G renamed ADC_V_I-
- net SNG-3F renamed ADC_W_I+
- net SNG-3G renamed ADC_W_I-
- net SNG-4F renamed ADC_BAT_I+
- net SNG-4G renamed ADC_BAT_I-
- net SNG-V1+ renamed ADC_U_V+
- net SNG-V1- renamed ADC_U_V-
- net SNG-V2+ renamed ADC_V_V+
- net SNG-V2- renamed ADC_V_V-
- net SNG-V3+ renamed ADC_W_V+
- net SNG-V3- renamed ADC_W_V-
- net SNG-V4+ renamed ADC_BAT_V+
- net SNG-V4- renamed ADC_BAT_V-
- no-connect marks 0 -> 4
Other:
- note added: "AD7606C-18 datasheet (Rev. B)"
- note removed: "AD7606C-18 datasheet (Rev. A)"

Commit message: Add 100 Ohm series resistors on the J4 lines, bottom side
RN1, RN2 (R_Array_Concave_4x0603, the 4 x 100 Ohm array of OPEN_WEIGHT)
and R39-R41 (0603) sit inline on the existing B.Cu buses between IC1 and
J4; only the bus sections around them were redrawn. Element order follows
the routing: RN2 = DOUTD..DOUTA, R41 = SDI, RN1 = FRSTDATA, SCLK, CS,
BUSY, R40 = RESET, R39 = CONVST. J4 pinout unchanged.

Schematic: IC1 keeps its wires with local labels (IC side); the resistor
block carries the ADC_* global labels (J4 side). TP15 / TP16 move to the
IC side, where their pads are on the board.

Fixes a short: the +5VA via of R36 (138.6, 60.2) sat on the ADC_~{CS}
track; bus B now passes above it.

DRC 206 -> 203 (the short's 3 errors), parity 34 -> 16 (all pre-existing),
ERC unchanged; top and inner layers identical.

Co-Authored-By: Claude Opus 5.5 <noreply@anthropic.com>
Parts:
- added R39, R40, R41: 100Ω, OPEN_PHASE:R_0603_1608Metric, symbol OPEN_PHASE:R
- added RN1, RN2: RP_100Ω, OPEN_PHASE:R_Array_Concave_4x0603, symbol OPEN_PHASE:R_Pack04
Connections:
- net ADC_BUSY: now also RN1.5 (R4.2); no longer IC1.14 (BUSY), TP16.1
- net ADC_CONVST: now also R39.2; no longer IC1.9 (CONVST), TP15.1
- net ADC_DOUTA: now also RN2.5 (R4.2); no longer IC1.24 (DB9/DOUTA)
- net ADC_DOUTB: now also RN2.6 (R3.2); no longer IC1.25 (DB10/DOUTB)
- net ADC_DOUTC: now also RN2.7 (R2.2); no longer IC1.27 (DB11/DOUTC)
- net ADC_DOUTD: now also RN2.8 (R1.2); no longer IC1.28 (DB12/DOUTD)
- net ADC_FRSTDATA: now also RN1.8 (R1.2); no longer IC1.15 (FRSTDATA)
- net ADC_RESET: now also R40.2; no longer IC1.11 (RESET)
- net ADC_SCLK: now also RN1.7 (R2.2); no longer IC1.12 (~{RD}/SCLK)
- net ADC_SDI: now also R41.2; no longer IC1.29 (DB13/SDI)
- net ADC_~{CS}: now also RN1.6 (R3.2); no longer IC1.13 (~{CS})
- new net BUSY: IC1.14 (BUSY), RN1.4 (R4.1), TP16.1
- new net CONVST: IC1.9 (CONVST), R39.1, TP15.1
- new net DOUTA: IC1.24 (DB9/DOUTA), RN2.4 (R4.1)
- new net DOUTB: IC1.25 (DB10/DOUTB), RN2.3 (R3.1)
- new net DOUTC: IC1.27 (DB11/DOUTC), RN2.2 (R2.1)
- new net DOUTD: IC1.28 (DB12/DOUTD), RN2.1 (R1.1)
- new net FRSTDATA: IC1.15 (FRSTDATA), RN1.1 (R1.1)
- new net RESET: IC1.11 (RESET), R40.1
- new net SCLK: IC1.12 (~{RD}/SCLK), RN1.2 (R2.1)
- new net SDI: IC1.29 (DB13/SDI), R41.1
- new net ~{CS}: IC1.13 (~{CS}), RN1.3 (R3.1)

Commit message: Add 100k pull-up on ADC CS and pull-downs on CONVST and RESET
R42 (CS to +3.3V), R43 (CONVST to GND) and R44 (RESET to GND), 100k 0603
on the AD7606C side, as R8 on OPEN_WEIGHT: the lines stay in a known state
while the host does not drive them (MCU in reset, wire unplugged).

Bottom side: R43 and R44 go straight into the B.Cu GND pour; R44 sits at
the east end of the BUSY / RESET band so the band stays connected. R42
reaches +3.3V through a new via at (165.8, 64.7) into the In2 +3.3V
branch, under the IC1 corner (only that via's clearance changes on F.Cu
and In1).

DRC 203 = 203, unconnected 4 = 4, parity 16 = 16, ERC unchanged.

Co-Authored-By: Claude Opus 5.5 <noreply@anthropic.com>
Parts:
- added R42, R43, R44: 100kΩ, OPEN_PHASE:R_0603_1608Metric, symbol OPEN_PHASE:R
Connections:
- net +3.3V: now also R42.1
- net CONVST: now also R43.1
- net GND: now also R43.2, R44.2
- net RESET: now also R44.1
- net ~{CS}: now also R42.2
